File: Hardware/PCB-design/Lipmouse_Teensy/Lipmouse_Teensy.sch (EAGLE design)
At the start: 24 parts, among them IC1 24FC1025-I/P, Q1 BS170, X1 1503_02, X2 1503_02

Commit message: Update design, update BOM to new version
Parts:
- RN1: value 390R -> 220R
- renumbered U$3 to U3
Changed lines of the file:
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@@
 <grid distance="0.1" unitdist="inch" unit="inch" style="lines" multiple="1" display="no" altdistance="0.01" altunitdist="inch" altunit="inch"/>
 <layers>
-<layer number="1" name="Top" color="4" fill="1" visible="no" active="no"/>
-<layer number="16" name="Bottom" color="1" fill="1" visible="no" active="no"/>
-<layer number="17" name="Pads" color="2" fill="1" visible="no" active="no"/>
-<layer number="18" name="Vias" color="2" fill="1" visible="no" active="no"/>
-<layer number="19" name="Unrouted" color="6" fill="1" visible="no" active="no"/>
-<layer number="20" name="Dimension" color="15" fill="1" visible="no" active="no"/>
-<layer number="21" name="tPlace" color="7" fill="1" visible="no" active="no"/>
-<layer number="22" name="bPlace" color="7" fill="1" visible="no" active="no"/>
-<layer number="23" name="tOrigins" color="15" fill="1" visible="no" active="no"/>
-<layer number="24" name="bOrigins" color="15" fill="1" visible="no" active="no"/>
-<layer number="25" name="tNames" color="7" fill="1" visible="no" active="no"/>
-<layer number="26" name="bNames" color="7" fill="1" visible="no" active="no"/>
-<layer number="27" name="tValues" color="7" fill="1" visible="no" active="no"/>
-<layer number="28" name="bValues" color="7" fill="1" visible="no" active="no"/>
+<layer number="1" name="Top" color="4" fill="1" visible="yes" active="no"/>
+<layer number="16" name="Bottom" color="1" fill="1" visible="yes" active="no"/>
+<layer number="17" name="Pads" color="2" fill="1" visible="yes" active="no"/>
+<layer number="18" name="Vias" color="2" fill="1" visible="yes" active="no"/>
+<layer number="19" name="Unrouted" color="6" fill="1" visible="yes" active="no"/>
+<layer number="20" name="Dimension" color="15" fill="1" visible="yes" active="no"/>
+<layer number="21" name="tPlace" color="7" fill="1" visible="yes" active="no"/>
+<layer number="22" name="bPlace" color="7" fill="1" visible="yes" active="no"/>
+<layer number="23" name="tOrigins" color="15" fill="1" visible="yes" active="no"/>
+<layer number="24" name="bOrigins" color="15" fill="1" visible="yes" active="no"/>
+<layer number="25" name="tNames" color="7" fill="1" visible="yes" active="no"/>
+<layer number="26" name="bNames" color="7" fill="1" visible="yes" active="no"/>
+<layer number="27" name="tValues" color="7" fill="1" visible="yes" active="no"/>
+<layer number="28" name="bValues" color="7" fill="1" visible="yes" active="no"/>
 <layer number="29" name="tStop" color="7" fill="3" visible="no" active="no"/>
 <layer number="30" name="bStop" color="7" fill="6" visible="no" active="no"/>
@@
 <layer number="35" name="tGlue" color="7" fill="4" visible="no" active="no"/>
 <layer number="36" name="bGlue" color="7" fill="5" visible="no" active="no"/>
-<layer number="37" name="tTest" color="7" fill="1" visible="no" active="no"/>
-<layer number="38" name="bTest" color="7" fill="1" visible="no" active="no"/>
+<layer number="37" name="tTest" color="7" fill="1" visible="yes" active="no"/>
+<layer number="38" name="bTest" color="7" fill="1" visible="yes" active="no"/>
 <layer number="39" name="tKeepout" color="4" fill="11" visible="no" active="no"/>
 <layer number="40" name="bKeepout" color="1" fill="11" visible="no" active="no"/>
@@
 <layer number="44" name="Drills" color="7" fill="1" visible="no" active="no"/>
 <layer number="45" name="Holes" color="7" fill="1" visible="no" active="no"/>
-<layer number="46" name="Milling" color="3" fill="1" visible="no" active="no"/>
-<layer number="47" name="Measures" color="7" fill="1" visible="no" active="no"/>
-<layer number="48" name="Document" color="7" fill="1" visible="no" active="no"/>
-<layer number="49" name="Reference" color="7" fill="1" visible="no" active="no"/>
-<layer number="50" name="dxf" color="7" fill="1" visible="no" active="no"/>
-<layer number="51" name="tDocu" color="7" fill="1" visible="no" active="no"/>
-<layer number="52" name="bDocu" color="7" fill="1" visible="no" active="no"/>
-<layer number="53" name="tGND_GNDA" color="7" fill="9" visible="no" active="no"/>
-<layer number="54" name="bGND_GNDA" color="1" fill="9" visible="no" active="no"/>
-<layer number="56" name="wert" color="7" fill="1" visible="no" active="no"/>
-<layer number="57" name="tCAD" color="7" fill="1" visible="no" active="no"/>
-<layer number="60" name="Board" color="7" fill="1" visible="no" active="no"/>
+<layer number="46" name="Milling" color="3" fill="1" visible="yes" active="no"/>
+<layer number="47" name="Measures" color="7" fill="1" visible="yes" active="no"/>
+<layer number="48" name="Document" color="7" fill="1" visible="yes" active="no"/>
+<layer number="49" name="Reference" color="7" fill="1" visible="yes" active="no"/>
+<layer number="50" name="dxf" color="7" fill="1" visible="yes" active="no"/>
+<layer number="51" name="tDocu" color="7" fill="1" visible="yes" active="no"/>
+<layer number="52" name="bDocu" color="7" fill="1" visible="yes" active="no"/>
+<layer number="53" name="tGND_GNDA" color="7" fill="9" visible="yes" active="no"/>
+<layer number="54" name="bGND_GNDA" color="1" fill="9" visible="yes" active="no"/>
+<layer number="56" name="wert" color="7" fill="1" visible="yes" active="no"/>
+<layer number="57" name="tCAD" color="7" fill="1" visible="yes" active="no"/>
+<layer number="60" name="Board" color="7" fill="1" visible="yes" active="no"/>
 <layer number="91" name="Nets" color="2" fill="1" visible="yes" active="yes"/>
 <layer number="92" name="Busses" color="1" fill="1" visible="yes" active="yes"/>
@@
 <part name="GND9" library="supply1" deviceset="GND" device=""/>
 <part name="LED5" library="led" deviceset="LED" device="5MM" value="TSAL6200"/>
-<part name="U$3" library="TSOPXXXX" deviceset="TSOP48XX" device="" value="TSOP4838"/>
+<part name="U3" library="TSOPXXXX" deviceset="TSOP48XX" device="" value="TSOP4838"/>
 <part name="P+7" library="supply1" deviceset="VCC" device=""/>
 <part name="GND10" library="supply1" deviceset="GND" device=""/>
@@
 <part name="C1" library="resistor" deviceset="C-EU" device="025-025X050" value="100nF"/>
 <part name="C2" library="resistor" deviceset="C-EU" device="025-025X050" value="100nF"/>
-<part name="RN1" library="resistor-net" deviceset="RN04" device="" value="390R"/>
+<part name="RN1" library="resistor-net" deviceset="RN04" device="" value="220R"/>
 <part name="RN2" library="resistor-net" deviceset="RN04" device="" value="10k"/>
 <part name="R11" library="resistor" deviceset="R-EU_" device="0309/V" value="120R"/>
@@
 <attribute name="VALUE" x="59.055" y="167.132" size="1.778" layer="96" rot="MR270"/>
 </instance>
-<instance part="U$3" gate="G$1" x="12.7" y="157.48"/>
+<instance part="U3" gate="G$1" x="12.7" y="157.48"/>
 <instance part="P+7" gate="VCC" x="22.86" y="167.64" smashed="yes">
 <attribute name="VALUE" x="22.86" y="170.18" size="1.778" layer="96" rot="R90"/>
@@
 </segment>
 <segment>
-<pinref part="U$3" gate="G$1" pin="GND"/>
+<pinref part="U3" gate="G$1" pin="GND"/>
 <wire x1="17.78" y1="154.94" x2="22.86" y2="154.94" width="0.1524" layer="91"/>
 <wire x1="22.86" y1="154.94" x2="22.86" y2="152.4" width="0.1524" layer="91"/>
@@
 </segment>
 <segment>
-<pinref part="U$3" gate="G$1" pin="VCC"/>
+<pinref part="U3" gate="G$1" pin="VCC"/>
 <wire x1="17.78" y1="160.02" x2="22.86" y2="160.02" width="0.1524" layer="91"/>
 <wire x1="22.86" y1="160.02" x2="22.86" y2="165.1" width="0.1524" layer="91"/>
@@
 <net name="TSOP" class="0">
 <segment>
-<pinref part="U$3" gate="G$1" pin="OUT"/>
+<pinref part="U3" gate="G$1" pin="OUT"/>
 <wire x1="17.78" y1="157.48" x2="27.94" y2="157.48" width="0.1524" layer="91"/>
 <label x="20.32" y="157.48" size="1.778" layer="95"/>

Commit message: Update to PCB version 2.
Using TeensyLC now, with through hole parts only (easier to solder without experience)
Parts:
- renumbered U$1 to U1, U$2 to U2

Commit message: Update readme Changed PCB, added a buzzer. Should be final for rev2.5
Parts:
- added R3: 10k, resistor:R-EU_0309/V
- added SG1: RS: 457011, buzzer:EFBAA40D101
Connections:
- new net N$5: R3.1, SG1.1
- new net PIEZO: R3.2, U1.9/RX2/PWM
- net GND: now also SG1.2
- net SDA_EEPROM: now also R2.2; no longer R2.1
- net VCC: now also R2.1; no longer R2.2
Other:
- moved on the sheet: R2
Changed lines of the file:
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@@
 <part name="GND5" library="supply1" deviceset="GND" device=""/>
 <part name="I2C" library="pinhead" deviceset="PINHD-1X2" device=""/>
+<part name="SG1" library="buzzer" deviceset="EFB?" device="AA40D101" value="RS: 457011"/>
+<part name="R3" library="resistor" deviceset="R-EU_" device="0309/V" value="10k"/>
+<part name="GND6" library="supply1" deviceset="GND" device=""/>
 </parts>
 <sheets>
@@
 <plain>
 <wire x1="154.94" y1="2.54" x2="81.28" y2="2.54" width="0.1524" layer="97"/>
-<wire x1="81.28" y1="2.54" x2="81.28" y2="53.34" width="0.1524" layer="97"/>
-<wire x1="81.28" y1="53.34" x2="157.48" y2="53.34" width="0.1524" layer="97"/>
-<wire x1="157.48" y1="53.34" x2="157.48" y2="2.54" width="0.1524" layer="97"/>
-<text x="83.82" y="48.26" size="1.778" layer="97">EEPROM</text>
-<wire x1="76.2" y1="53.34" x2="2.54" y2="53.34" width="0.1524" layer="97"/>
-<wire x1="2.54" y1="53.34" x2="2.54" y2="2.54" width="0.1524" layer="97"/>
+<wire x1="81.28" y1="2.54" x2="81.28" y2="58.42" width="0.1524" layer="97"/>
+<wire x1="81.28" y1="58.42" x2="157.48" y2="58.42" width="0.1524" layer="97"/>
+<wire x1="157.48" y1="58.42" x2="157.48" y2="2.54" width="0.1524" layer="97"/>
+<text x="83.82" y="53.34" size="1.778" layer="97">EEPROM</text>
+<wire x1="76.2" y1="58.42" x2="2.54" y2="58.42" width="0.1524" layer="97"/>
+<wire x1="2.54" y1="58.42" x2="2.54" y2="2.54" width="0.1524" layer="97"/>
 <wire x1="2.54" y1="2.54" x2="76.2" y2="2.54" width="0.1524" layer="97"/>
-<wire x1="76.2" y1="2.54" x2="76.2" y2="53.34" width="0.1524" layer="97"/>
-<text x="5.08" y="48.26" size="1.778" layer="97">Pressure Sensor</text>
+<wire x1="76.2" y1="2.54" x2="76.2" y2="58.42" width="0.1524" layer="97"/>
+<text x="5.08" y="53.34" size="1.778" layer="97">Pressure Sensor</text>
 <text x="30.48" y="5.08" size="1.778" layer="97">additional mounting
 stability (NC)</text>
@@
 <text x="5.08" y="134.62" size="1.778" layer="97">IR receiver/transmitter</text>
 <wire x1="2.54" y1="124.46" x2="76.2" y2="124.46" width="0.1524" layer="97"/>
-<wire x1="76.2" y1="124.46" x2="76.2" y2="60.96" width="0.1524" layer="97"/>
-<wire x1="76.2" y1="60.96" x2="2.54" y2="60.96" width="0.1524" layer="97"/>
-<wire x1="2.54" y1="60.96" x2="2.54" y2="124.46" width="0.1524" layer="97"/>
+<wire x1="76.2" y1="124.46" x2="76.2" y2="63.5" width="0.1524" layer="97"/>
+<wire x1="76.2" y1="63.5" x2="2.54" y2="63.5" width="0.1524" layer="97"/>
+<wire x1="2.54" y1="63.5" x2="2.54" y2="124.46" width="0.1524" layer="97"/>
 <text x="5.08" y="66.04" size="1.778" layer="97">Push-Buttons
 External Buttons</text>
@@
 -) Full serial port
 -) I2C from EEPROM</text>
+<wire x1="160.02" y1="58.42" x2="193.04" y2="58.42" width="0.1524" layer="97"/>
+<wire x1="193.04" y1="58.42" x2="193.04" y2="38.1" width="0.1524" layer="97"/>
+<wire x1="193.04" y1="38.1" x2="160.02" y2="38.1" width="0.1524" layer="97"/>
+<wire x1="160.02" y1="38.1" x2="160.02" y2="58.42" width="0.1524" layer="97"/>
 </plain>
 <instances>
@@
 <instance part="GND3" gate="1" x="63.5" y="137.16"/>
 <instance part="R1" gate="G$1" x="101.6" y="33.02" rot="R90"/>
-<instance part="R2" gate="G$1" x="142.24" y="33.02" rot="R90"/>
+<instance part="R2" gate="G$1" x="142.24" y="30.48" rot="R270"/>
 <instance part="P+1" gate="VCC" x="129.54" y="45.72"/>
 <instance part="X1" gate="G$1" x="48.26" y="109.22" rot="R180"/>
@@
 </instance>
 <instance part="I2C" gate="G$1" x="231.14" y="144.78"/>
+<instance part="SG1" gate="G$1" x="180.34" y="48.26" smashed="yes">
+<attribute name="NAME" x="172.72" y="54.61" size="1.778" layer="95"/>
+<attribute name="VALUE" x="179.07" y="55.88" size="1.778" layer="96"/>
+</instance>
+<instance part="R3" gate="G$1" x="170.18" y="45.72" rot="R180"/>
+<instance part="GND6" gate="1" x="187.96" y="43.18"/>
 </instances>
 <busses>
@@
 <pinref part="GND5" gate="1" pin="GND"/>
 </segment>
+<segment>
+<pinref part="SG1" gate="G$1" pin="2"/>
+<wire x1="185.42" y1="45.72" x2="187.96" y2="45.72" width="0.1524" layer="91"/>
+<pinref part="GND6" gate="1" pin="GND"/>
+</segment>
 </net>
 <net name="FSR1" class="0">
@@
 <wire x1="101.6" y1="38.1" x2="101.6" y2="40.64" width="0.1524" layer="91"/>
 <wire x1="101.6" y1="40.64" x2="129.54" y2="40.64" width="0.1524" layer="91"/>
-<pinref part="R2" gate="G$1" pin="2"/>
 <wire x1="129.54" y1="40.64" x2="142.24" y2="40.64" width="0.1524" layer="91"/>
-<wire x1="142.24" y1="40.64" x2="142.24" y2="38.1" width="0.1524" layer="91"/>
 <pinref part="IC1" gate="G$1" pin="VCC"/>
 <wire x1="129.54" y1="33.02" x2="129.54" y2="40.64" width="0.1524" layer="91"/>
@@
 <wire x1="129.54" y1="40.64" x2="129.54" y2="43.18" width="0.1524" layer="91"/>
 <pinref part="P+1" gate="VCC" pin="VCC"/>
+<pinref part="R2" gate="G$1" pin="1"/>
+<wire x1="142.24" y1="35.56" x2="142.24" y2="40.64" width="0.1524" layer="91"/>
 </segment>
 <segment>
@@
 <pinref part="IC1" gate="G$1" pin="SDA"/>
 <wire x1="137.16" y1="20.32" x2="142.24" y2="20.32" width="0.1524" layer="91"/>
-<pinref part="R2" gate="G$1" pin="1"/>
+<label x="139.7" y="17.78" size="1.778" layer="95"/>
+<pinref part="R2" gate="G$1" pin="2"/>
 <wire x1="142.24" y1="20.32" x2="152.4" y2="20.32" width="0.1524" layer="91"/>
-<wire x1="142.24" y1="27.94" x2="142.24" y2="20.32" width="0.1524" layer="91"/>
-<junction x="142.24" y="20.32"/>
-<label x="139.7" y="17.78" size="1.778" layer="95"/>
+<wire x1="142.24" y1="25.4" x2="142.24" y2="20.32" width="0.1524" layer="91"/>
 </segment>
 <segment>
@@
 </segment>
 </net>
+<net name="PIEZO" class="0">
+<segment>
+<pinref part="R3" gate="G$1" pin="2"/>
+<wire x1="165.1" y1="45.72" x2="165.1" y2="55.88" width="0.1524" layer="91"/>
+<label x="165.1" y="45.72" size="1.778" layer="95" rot="R90"/>
+</segment>
+<segment>
+<pinref part="U1" gate="G$1" pin="9/RX2/PWM"/>
+<wire x1="104.14" y1="127" x2="116.84" y2="127" width="0.1524" layer="91"/>
+<label x="104.14" y="127" size="1.778" layer="95"/>
+</segment>
+</net>
+<net name="N$5" class="0">
+<segment>
+<pinref part="R3" gate="G$1" pin="1"/>
+<pinref part="SG1" gate="G$1" pin="1"/>
+<wire x1="175.26" y1="45.72" x2="177.8" y2="45.72" width="0.1524" layer="91"/>
+</segment>
+</net>

Commit message: Updated PCB: changed Gate series resistor into pull-down (avoiding floating gates if Teensy is not programmed)
Parts:
- R1, R2, R3: value 10k -> 4k7
- R11: value 120R -> 4k7
- R12: value 22R -> 12R
Connections:
- removed net N$8: Q1.G, R11.2
- net GND: now also R11.1
- net IRLED: now also Q1.G, R11.2; no longer R11.1
Other:
- moved on the sheet: R11
Changed lines of the file:
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@@
 <?xml version="1.0" encoding="utf-8"?>
 <!DOCTYPE eagle SYSTEM "eagle.dtd">
-<eagle version="6.6.0">
+<eagle version="7.5.0">
 <drawing>
 <settings>
@@
 <part name="RN1" library="resistor-net" deviceset="RN04" device="" value="220R"/>
 <part name="RN2" library="resistor-net" deviceset="RN04" device="" value="10k"/>
-<part name="R11" library="resistor" deviceset="R-EU_" device="0309/V" value="120R"/>
+<part name="R11" library="resistor" deviceset="R-EU_" device="0309/V" value="4k7"/>
 <part name="Q1" library="transistor-small-signal" deviceset="BS170" device=""/>
 <part name="IC1" library="microchip" deviceset="24*" device="P" technology="LC256" value="24FC1025-I/P"/>
 <part name="U1" library="Teensy_3_Series_Board_v1.0" deviceset="TEENSY_3.1_BASIC" device=""/>
-<part name="R12" library="resistor" deviceset="R-EU_" device="0309/V" value="22R"/>
+<part name="R12" library="resistor" deviceset="R-EU_" device="0309/V" value="12R"/>
 <part name="GND13" library="supply1" deviceset="GND" device=""/>
 <part name="GND2" library="supply1" deviceset="GND" device=""/>
 <part name="GND3" library="supply1" deviceset="GND" device=""/>
-<part name="R1" library="resistor" deviceset="R-EU_" device="0309/V" value="10k"/>
-<part name="R2" library="resistor" deviceset="R-EU_" device="0309/V" value="10k"/>
+<part name="R1" library="resistor" deviceset="R-EU_" device="0309/V" value="4k7"/>
+<part name="R2" library="resistor" deviceset="R-EU_" device="0309/V" value="4k7"/>
 <part name="P+1" library="supply1" deviceset="VCC" device=""/>
 <part name="X1" library="con-lumberg" deviceset="1503_02" device=""/>
@@
 <part name="I2C" library="pinhead" deviceset="PINHD-1X2" device=""/>
 <part name="SG1" library="buzzer" deviceset="EFB?" device="AA40D101" value="RS: 457011"/>
-<part name="R3" library="resistor" deviceset="R-EU_" device="0309/V" value="10k"/>
+<part name="R3" library="resistor" deviceset="R-EU_" device="0309/V" value="4k7"/>
 <part name="GND6" library="supply1" deviceset="GND" device=""/>
+<part name="GND7" library="supply1" deviceset="GND" device=""/>
 </parts>
 <sheets>
@@
 stability (NC)</text>
 <wire x1="2.54" y1="177.8" x2="76.2" y2="177.8" width="0.1524" layer="97"/>
-<wire x1="76.2" y1="177.8" x2="76.2" y2="132.08" width="0.1524" layer="97"/>
-<wire x1="76.2" y1="132.08" x2="2.54" y2="132.08" width="0.1524" layer="97"/>
-<wire x1="2.54" y1="132.08" x2="2.54" y2="177.8" width="0.1524" layer="97"/>
-<text x="5.08" y="134.62" size="1.778" layer="97">IR receiver/transmitter</text>
+<wire x1="76.2" y1="177.8" x2="76.2" y2="127" width="0.1524" layer="97"/>
+<wire x1="76.2" y1="127" x2="2.54" y2="127" width="0.1524" layer="97"/>
+<wire x1="2.54" y1="127" x2="2.54" y2="177.8" width="0.1524" layer="97"/>
+<text x="5.08" y="129.54" size="1.778" layer="97">IR receiver/transmitter</text>
 <wire x1="2.54" y1="124.46" x2="76.2" y2="124.46" width="0.1524" layer="97"/>
 <wire x1="76.2" y1="124.46" x2="76.2" y2="63.5" width="0.1524" layer="97"/>
@@
 <instance part="RN1" gate="1" x="228.6" y="129.54"/>
 <instance part="RN2" gate="1" x="220.98" y="76.2"/>
-<instance part="R11" gate="G$1" x="50.8" y="144.78"/>
+<instance part="R11" gate="G$1" x="53.34" y="139.7" rot="R90"/>
 <instance part="Q1" gate="1" x="60.96" y="144.78"/>
 <instance part="IC1" gate="G$1" x="121.92" y="20.32"/>
@@
 <instance part="R3" gate="G$1" x="170.18" y="45.72" rot="R180"/>
 <instance part="GND6" gate="1" x="187.96" y="43.18"/>
+<instance part="GND7" gate="1" x="53.34" y="132.08"/>
 </instances>
 <busses>
@@
 <pinref part="GND6" gate="1" pin="GND"/>
 </segment>
+<segment>
+<pinref part="R11" gate="G$1" pin="1"/>
+<pinref part="GND7" gate="1" pin="GND"/>
+</segment>
 </net>
 <net name="FSR1" class="0">
@@
 </segment>
 </net>
-<net name="N$8" class="0">
-<segment>
-<pinref part="R11" gate="G$1" pin="2"/>
-<pinref part="Q1" gate="1" pin="G"/>
-</segment>
-</net>
 <net name="N$9" class="0">
 <segment>
@@
 <net name="IRLED" class="0">
 <segment>
-<pinref part="R11" gate="G$1" pin="1"/>
-<wire x1="45.72" y1="144.78" x2="35.56" y2="144.78" width="0.1524" layer="91"/>
-<label x="35.56" y="144.78" size="1.778" layer="95"/>
-</segment>
-<segment>
 <pinref part="U1" gate="G$1" pin="6/PWM"/>
 <wire x1="116.84" y1="134.62" x2="104.14" y2="134.62" width="0.1524" layer="91"/>
 <label x="104.14" y="134.62" size="1.778" layer="95"/>
 </segment>
-</net>
+<segment>
+<pinref part="R11" gate="G$1" pin="2"/>
+<pinref part="Q1" gate="1" pin="G"/>
+<wire x1="53.34" y1="144.78" x2="55.88" y2="144.78" width="0.1524" layer="91"/>
+<wire x1="53.34" y1="144.78" x2="38.1" y2="144.78" width="0.1524" layer="91"/>
+<label x="38.1" y="144.78" size="1.778" layer="95"/>
+</segment>
+</net>
