File: Hardware/PCB-design/sensorboard/RES-DMS-NAU7802.kicad_pcb (KiCad board)
At the start: 2 copper layers, 32 x 32 mm, 43 parts, among them J1 Conn_01x06, J2 straingauge, J4 straingauge, J5 straingauge, J6 straingauge, U1 NAU7802-SGI

Commit message: Changed resistor values of half bridge (not sensing; should be resistor network)
Parts:
- R11, R12, R13, R14: value 1k -> 555R
Changed lines of the file:
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@@
       (effects (font (size 0.7 0.7) (thickness 0.12)))
     )
-    (fp_text value "1k" (at 0 1.82) (layer "F.Fab")
+    (fp_text value "555R" (at 0 1.82) (layer "F.Fab")
       (effects (font (size 1 1) (thickness 0.15)))
     )
@@
       (effects (font (size 0.7 0.7) (thickness 0.12)))
     )
-    (fp_text value "1k" (at 0 1.82) (layer "F.Fab")
+    (fp_text value "555R" (at 0 1.82) (layer "F.Fab")
       (effects (font (size 1 1) (thickness 0.15)))
     )
@@
       (effects (font (size 0.7 0.7) (thickness 0.12)))
     )
-    (fp_text value "1k" (at 0 1.82) (layer "F.Fab")
+    (fp_text value "555R" (at 0 1.82) (layer "F.Fab")
       (effects (font (size 1 1) (thickness 0.15)))
     )
@@
       (effects (font (size 0.7 0.7) (thickness 0.12)))
     )
-    (fp_text value "1k" (at 0 1.82) (layer "F.Fab")
+    (fp_text value "555R" (at 0 1.82) (layer "F.Fab")
       (effects (font (size 1 1) (thickness 0.15)))
     )

Commit message: Updated schematic/PCB (values for R-Net or alternatives), updated iBOM
Parts:
- R10, R7, R8, R9: value 1k -> DNP (1k RMCF)
- R11, R12, R13, R14: value 555R -> DNP (1k)
- RN1: value R_Pack04 -> CAY16-1001F4LF
