File: Hardware/PCB-design/sensorboard_MPRLS/sensorboard_MPRLS.kicad_pcb (KiCad board)
At the start: 2 copper layers, 15 x 14.7 mm, 13 parts, among them J1 Conn_01x01, J2 Conn_01x01, J3 Conn_01x01, J4 Conn_01x01, J5 Conn_01x01, U1 MPRLS0025PA00001AB

Commit message: MPRLS board 0.9mm smaller, does not fit in edge connector
Routing:
- net GND: track 6.79 -> 13.9 mm, vias 16 -> 18
- net VCC: track 26.0 -> 27.8 mm, vias 3 -> 4
Other:
- outline, holes or cut-outs redrawn
Changed lines of the file:
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@@
   (gr_line (start 130 130) (end 145 130)
     (stroke (width 0.1) (type default)) (layer "Edge.Cuts"))
-  (gr_line (start 142.9 115.7) (end 142.9 120)
+  (gr_line (start 142.3 115.7) (end 142.3 120)
     (stroke (width 0.1) (type default)) (layer "Edge.Cuts"))
-  (gr_line (start 132.5 115.3) (end 132.1 115.7)
+  (gr_line (start 133.1 115.3) (end 132.7 115.7)
     (stroke (width 0.1) (type default)) (layer "Edge.Cuts"))
   (gr_line (start 145 130) (end 145 120)
     (stroke (width 0.1) (type default)) (layer "Edge.Cuts"))
-  (gr_line (start 142.9 120) (end 145 120)
+  (gr_line (start 142.3 120) (end 145 120)
     (stroke (width 0.1) (type default)) (layer "Edge.Cuts"))
   (gr_line (start 130 130) (end 130 120)
     (stroke (width 0.1) (type default)) (layer "Edge.Cuts"))
-  (gr_line (start 130 120) (end 132.1 120)
+  (gr_line (start 130 120) (end 132.7 120)
     (stroke (width 0.1) (type default)) (layer "Edge.Cuts"))
-  (gr_line (start 142.5 115.3) (end 142.9 115.7)
+  (gr_line (start 141.9 115.3) (end 142.3 115.7)
     (stroke (width 0.1) (type default)) (layer "Edge.Cuts"))
-  (gr_line (start 132.5 115.3) (end 142.5 115.3)
+  (gr_line (start 133.1 115.3) (end 141.9 115.3)
     (stroke (width 0.1) (type default)) (layer "Edge.Cuts"))
-  (gr_line (start 132.1 120) (end 132.1 115.7)
+  (gr_line (start 132.7 120) (end 132.7 115.7)
     (stroke (width 0.1) (type default)) (layer "Edge.Cuts"))
   (gr_text "1u" (at 132.7 125.7 90) (layer "B.SilkS")
@@
     (effects (font (size 0.5 0.5) (thickness 0.125) bold) (justify left bottom))
   )
+  (segment (start 136.4 118.6) (end 136.4 120.2) (width 0.3) (layer "F.Cu") (net 1))
   (segment (start 140.605 127.57) (end 141.2 126.975) (width 0.3) (layer "F.Cu") (net 1))
   (segment (start 144.1125 121.7) (end 144.1125 122.5) (width 0.3) (layer "F.Cu") (net 1))
   (segment (start 141.9 127.9) (end 141.9 126.975) (width 0.3) (layer "F.Cu") (net 1))
+  (segment (start 135.5 117.7) (end 136.4 118.6) (width 0.3) (layer "F.Cu") (net 1))
   (segment (start 142.8 126.975) (end 141.9 126.975) (width 0.3) (layer "F.Cu") (net 1))
-  (segment (start 135.5 117.7) (end 135.5 119.5) (width 0.3) (layer "F.Cu") (net 1))
+  (segment (start 135.5 120.2) (end 135.5 119.5) (width 0.3) (layer "F.Cu") (net 1))
   (segment (start 141.9 126.975) (end 141.2 126.975) (width 0.3) (layer "F.Cu") (net 1))
+  (segment (start 135.5 119.5) (end 135.5 117.7) (width 0.3) (layer "F.Cu") (net 1))
   (segment (start 139.7 127.57) (end 140.605 127.57) (width 0.3) (layer "F.Cu") (net 1))
   (segment (start 144.2 123.7) (end 144.2 122.5875) (width 0.3) (layer "F.Cu") (net 1))
   (segment (start 144.2 122.5875) (end 144.1125 122.5) (width 0.3) (layer "F.Cu") (net 1))
   (segment (start 144.1125 120.9) (end 144.1125 121.7) (width 0.3) (layer "F.Cu") (net 1))
-  (segment (start 135.5 119.5) (end 134.8 120.2) (width 0.3) (layer "F.Cu") (net 1))
-  (via (at 134.8 120.2) (size 0.8) (drill 0.4) (layers "F.Cu" "B.Cu") (net 1))
+  (via (at 135.5 120.2) (size 0.8) (drill 0.4) (layers "F.Cu" "B.Cu") (net 1))
+  (via (at 136.4 120.2) (size 0.8) (drill 0.4) (layers "F.Cu" "B.Cu") (net 1))
   (via (at 144.2 123.7) (size 0.8) (drill 0.4) (layers "F.Cu" "B.Cu") (net 1))
   (via (at 141.9 127.9) (size 0.8) (drill 0.4) (layers "F.Cu" "B.Cu") (net 1))
@@
   (segment (start 142.2 127.6) (end 141.9 127.9) (width 0.3) (layer "B.Cu") (net 1))
   (segment (start 142.2 122.4) (end 142.2 123.4) (width 0.3) (layer "B.Cu") (net 1))
+  (segment (start 135.5 120.2) (end 136.4 120.2) (width 0.3) (layer "B.Cu") (net 1))
   (segment (start 143.9 123.4) (end 144.2 123.7) (width 0.3) (layer "B.Cu") (net 1))
-  (segment (start 134.8 120.2) (end 140 120.2) (width 0.3) (layer "B.Cu") (net 1))
   (segment (start 140 120.2) (end 142.2 122.4) (width 0.3) (layer "B.Cu") (net 1))
+  (segment (start 136.4 120.2) (end 140 120.2) (width 0.3) (layer "B.Cu") (net 1))
   (segment (start 142.2 123.4) (end 142.2 127.6) (width 0.3) (layer "B.Cu") (net 1))
+  (segment (start 133.5 119.4) (end 134.5 120.4) (width 0.3) (layer "F.Cu") (net 2))
+  (segment (start 133.5 119.6) (end 132.7 120.4) (width 0.3) (layer "F.Cu") (net 2))
+  (segment (start 133.5 120.3) (end 133.5 120.7) (width 0.3) (layer "F.Cu") (net 2))
+  (segment (start 133.5 120.7) (end 133.6 120.8) (width 0.3) (layer "F.Cu") (net 2))
   (segment (start 139.7 125.03) (end 140.805 125.03) (width 0.3) (layer "F.Cu") (net 2))
   (segment (start 140.805 125.03) (end 141.2 125.425) (width 0.3) (layer "F.Cu") (net 2))
+  (segment (start 133.5 117.7) (end 133.5 119.6) (width 0.3) (layer "F.Cu") (net 2))
+  (segment (start 133.5 117.7) (end 133.5 119.4) (width 0.3) (layer "F.Cu") (net 2))
   (segment (start 142.8 125.425) (end 141.2 125.425) (width 0.3) (layer "F.Cu") (net 2))
+  (segment (start 132.7 120.7) (end 132.6 120.8) (width 0.3) (layer "F.Cu") (net 2))
+  (segment (start 132.7 120.4) (end 132.7 120.7) (width 0.3) (layer "F.Cu") (net 2))
   (segment (start 133.5 117.7) (end 133.5 120.3) (width 0.3) (layer "F.Cu") (net 2))
   (segment (start 141.2 125.425) (end 141.2 124.5) (width 0.3) (layer "F.Cu") (net 2))
@@
   (via (at 141.2 124.5) (size 0.8) (drill 0.4) (layers "F.Cu" "B.Cu") (net 2))
   (via (at 130.5 125) (size 0.8) (drill 0.4) (layers "F.Cu" "B.Cu") (free) (net 2))
+  (via (at 132.6 120.8) (size 0.8) (drill 0.4) (layers "F.Cu" "B.Cu") (net 2))
   (via (at 133.5 129.5) (size 0.8) (drill 0.4) (layers "F.Cu" "B.Cu") (free) (net 2))
   (via (at 130.5 122) (size 0.8) (drill 0.4) (layers "F.Cu" "B.Cu") (free) (net 2))
@@
   (via (at 130.5 120.5) (size 0.8) (drill 0.4) (layers "F.Cu" "B.Cu") (free) (net 2))
   (via (at 130.5 129.5) (size 0.8) (drill 0.4) (layers "F.Cu" "B.Cu") (free) (net 2))
-  (via (at 133.5 120.3) (size 0.8) (drill 0.4) (layers "F.Cu" "B.Cu") (net 2))
+  (via (at 133.6 120.8) (size 0.8) (drill 0.4) (layers "F.Cu" "B.Cu") (net 2))
   (via (at 135 123.3) (size 0.8) (drill 0.4) (layers "F.Cu" "B.Cu") (free) (net 2))
   (via (at 132 129.5) (size 0.8) (drill 0.4) (layers "F.Cu" "B.Cu") (free) (net 2))
   (via (at 130.5 128) (size 0.8) (drill 0.4) (layers "F.Cu" "B.Cu") (free) (net 2))
+  (via (at 134.5 120.4) (size 0.8) (drill 0.4) (layers "F.Cu" "B.Cu") (net 2))
   (segment (start 135.5 127.57) (end 134.62 127.57) (width 0.25) (layer "F.Cu") (net 3))
   (segment (start 134.62 127.57) (end 134 126.95) (width 0.25) (layer "F.Cu") (net 3))

Commit message: Added iBOM for sensorboard, excluded edgeconnector from BOM
Parts:
- C4: value 1u -> 1u (optional, filter)
Changed lines of the file:
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@@
     (property "Sheetfile" "sensorboard_MPRLS.kicad_sch")
     (property "Sheetname" "")
+    (property "dnp" "")
     (property "ki_description" "Unpolarized capacitor")
     (property "ki_keywords" "cap capacitor")
@@
         (effects (font (size 0.5 0.5) (thickness 0.125) bold))
     )
-    (fp_text value "1u" (at 0 1.43 90) (layer "F.Fab")
+    (fp_text value "1u (optional, filter)" (at 0 1.43 90) (layer "F.Fab")
         (effects (font (size 0.5 0.5) (thickness 0.125)))
     )
@@
     (property "Sheetfile" "sensorboard_MPRLS.kicad_sch")
     (property "Sheetname" "")
+    (property "exclude_from_bom" "")
     (property "ki_description" "Generic connector, single row, 01x01, script generated (kicad-library-utils/schlib/autogen/connector/)")
     (property "ki_keywords" "connector")
-    (attr smd)
+    (attr smd exclude_from_bom)
     (fp_text reference "J5" (at 0 -0.5 unlocked) (layer "F.SilkS") hide
         (effects (font (size 0.5 0.5) (thickness 0.125)))
@@
     (property "Sheetfile" "sensorboard_MPRLS.kicad_sch")
     (property "Sheetname" "")
+    (property "exclude_from_bom" "")
     (property "ki_description" "Generic connector, single row, 01x01, script generated (kicad-library-utils/schlib/autogen/connector/)")
     (property "ki_keywords" "connector")
-    (attr smd)
+    (attr smd exclude_from_bom)
     (fp_text reference "J4" (at 0 -0.5 unlocked) (layer "F.SilkS") hide
         (effects (font (size 0.5 0.5) (thickness 0.125)))
@@
     (property "Sheetfile" "sensorboard_MPRLS.kicad_sch")
     (property "Sheetname" "")
+    (property "exclude_from_bom" "")
     (property "ki_description" "Generic connector, single row, 01x01, script generated (kicad-library-utils/schlib/autogen/connector/)")
     (property "ki_keywords" "connector")
-    (attr smd)
+    (attr smd exclude_from_bom)
     (fp_text reference "J1" (at 0 -0.5 unlocked) (layer "F.SilkS") hide
         (effects (font (size 0.5 0.5) (thickness 0.125)))
@@
     (property "Sheetfile" "sensorboard_MPRLS.kicad_sch")
     (property "Sheetname" "")
+    (property "exclude_from_bom" "")
     (property "ki_description" "Generic connector, single row, 01x01, script generated (kicad-library-utils/schlib/autogen/connector/)")
     (property "ki_keywords" "connector")
-    (attr smd)
+    (attr smd exclude_from_bom)
     (fp_text reference "J2" (at 0 -0.5 unlocked) (layer "F.SilkS") hide
         (effects (font (size 0.5 0.5) (thickness 0.125)))
@@
     (property "Sheetfile" "sensorboard_MPRLS.kicad_sch")
     (property "Sheetname" "")
+    (property "exclude_from_bom" "")
     (property "ki_description" "Generic connector, single row, 01x01, script generated (kicad-library-utils/schlib/autogen/connector/)")
     (property "ki_keywords" "connector")
-    (attr smd)
+    (attr smd exclude_from_bom)
     (fp_text reference "J3" (at 0 -0.5 unlocked) (layer "F.SilkS") hide
         (effects (font (size 0.5 0.5) (thickness 0.125)))
@@
     (property "Sheetfile" "sensorboard_MPRLS.kicad_sch")
     (property "Sheetname" "")
+    (property "exclude_from_bom" "")
     (property "ki_description" "3-pole Solder Jumper, pins 1+2 closed/bridged")
     (property "ki_keywords" "Solder Jumper SPDT")
-    (attr exclude_from_pos_files)
+    (attr exclude_from_pos_files exclude_from_bom)
     (net_tie_pad_groups "1, 2, 3")
     (fp_text reference "JP1" (at 0 -1.5 180 unlocked) (layer "F.SilkS")
