File: Hardware/PCB-design/sensorboard_DPS310/sensorboard_DPS310.kicad_sch (KiCad schematic)
At the start: 15 parts, among them J1 Conn_01x01, J2 Conn_01x01, J3 Conn_01x01, J4 Conn_01x01, J5 Conn_01x01, U2 DPS310

Commit message: Removed I2C addr. selection; removed holes and placed vias better.
Parts:
- removed H1, H2: ~, MountingHole:MountingHole_2.2mm_M2_Pad, symbol Mechanical:MountingHole_Pad
- removed R3: 10k, Resistor_SMD:R_0603_1608Metric_Pad0.98x0.95mm_HandSolder, symbol Device:R
Connections:
- no-connect marks 1 -> 2
Other:
- note removed: "If R3 is placed, the DPS310 has 0x76 as address, normal: 0x77"
Changed lines of the file:
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@@
   (junction (at 91.44 171.45) (diameter 0) (color 0 0 0 0)
   )
-  (junction (at 60.96 165.1) (diameter 0) (color 0 0 0 0)
-  )
   (junction (at 208.28 140.97) (diameter 0) (color 0 0 0 0)
   )
@@
   (junction (at 217.17 92.71) (diameter 0) (color 0 0 0 0)
   )
+  (no_connect (at 101.6 157.48))
   (no_connect (at 101.6 165.1))
-  (wire (pts (xy 60.96 165.1) (xy 64.77 165.1))
-    (stroke (width 0) (type default))
-  )
   (wire (pts (xy 91.44 171.45) (xy 91.44 173.355))
     (stroke (width 0) (type default))
@@
     (stroke (width 0) (type default))
   )
-  (wire (pts (xy 101.6 157.48) (xy 121.285 157.48))
-    (stroke (width 0) (type default))
-  )
   (wire (pts (xy 208.28 92.71) (xy 217.17 92.71))
     (stroke (width 0) (type default))
@@
     (stroke (width 0) (type default))
   )
-  (wire (pts (xy 121.285 157.48) (xy 121.285 160.02))
-    (stroke (width 0) (type default))
-  )
   (wire (pts (xy 88.9 171.45) (xy 91.44 171.45))
     (stroke (width 0) (type default))
   )
   (wire (pts (xy 208.28 133.35) (xy 219.71 133.35))
-    (stroke (width 0) (type default))
-  )
-  (wire (pts (xy 57.15 165.1) (xy 60.96 165.1))
     (stroke (width 0) (type default))
   )
@@
     (effects (font (size 1.27 1.27)) (justify left bottom))
   )
-  (text "If R3 is placed, the DPS310 has\n0x76 as address, normal: 0x77"
-    (at 108.585 155.575 0)
-    (effects (font (size 1.27 1.27)) (justify left bottom))
-  )
   (text "Landing pads for connector\n2mm spacing with cutouts"
     (at 148.59 69.85 0)
@@
     )
   )
-  (symbol (lib_id "power:GND") (at 121.285 167.64 0) (unit 1)
-    (in_bom yes) (on_board yes) (dnp no) (fields_autoplaced)
-    (property "Reference" "#PWR08" (at 121.285 173.99 0)
-      (effects (font (size 1.27 1.27)) hide)
-    )
-    (property "Value" "GND" (at 121.285 172.72 0)
-      (effects (font (size 1.27 1.27)))
-    )
-    (property "Footprint" "" (at 121.285 167.64 0)
-      (effects (font (size 1.27 1.27)) hide)
-    )
-    (property "Datasheet" "" (at 121.285 167.64 0)
-      (effects (font (size 1.27 1.27)) hide)
-    )
-    (pin "1")
-    (instances
-      (project "sensorboard_DPS310"
-        (path "/ed3d0d35-b5f6-4431-803a-14ff3cdab111"
-          (reference "#PWR08") (unit 1)
-        )
-      )
-    )
-  )
   (symbol (lib_id "Connector:TestPoint") (at 120.65 83.82 90) (unit 1)
     (in_bom yes) (on_board yes) (dnp no) (fields_autoplaced)
@@
         (path "/ed3d0d35-b5f6-4431-803a-14ff3cdab111"
           (reference "#FLG01") (unit 1)
-        )
-      )
-    )
-  )
-  (symbol (lib_id "power:GND") (at 60.96 165.1 0) (unit 1)
-    (in_bom yes) (on_board yes) (dnp no) (fields_autoplaced)
-    (property "Reference" "#PWR09" (at 60.96 171.45 0)
-      (effects (font (size 1.27 1.27)) hide)
-    )
-    (property "Value" "GND" (at 60.96 170.18 0)
-      (effects (font (size 1.27 1.27)))
-    )
-    (property "Footprint" "" (at 60.96 165.1 0)
-      (effects (font (size 1.27 1.27)) hide)
-    )
-    (property "Datasheet" "" (at 60.96 165.1 0)
-      (effects (font (size 1.27 1.27)) hide)
-    )
-    (pin "1")
-    (instances
-      (project "sensorboard_DPS310"
-        (path "/ed3d0d35-b5f6-4431-803a-14ff3cdab111"
-          (reference "#PWR09") (unit 1)
-        )
-      )
-    )
-  )
-  (symbol (lib_id "Mechanical:MountingHole_Pad") (at 57.15 162.56 0) (unit 1)
-    (in_bom yes) (on_board yes) (dnp no) (fields_autoplaced)
-    (property "Reference" "H1" (at 59.69 160.0779 0)
-      (effects (font (size 1.27 1.27)) (justify left))
-    )
-    (property "Value" "~" (at 59.69 162.5021 0)
-      (effects (font (size 1.27 1.27)) (justify left))
-    )
-    (property "Footprint" "MountingHole:MountingHole_2.2mm_M2_Pad" (at 57.15 162.56 0)
-      (effects (font (size 1.27 1.27)) hide)
-    )
-    (property "Datasheet" "~" (at 57.15 162.56 0)
-      (effects (font (size 1.27 1.27)) hide)
-    )
-    (pin "1")
-    (instances
-      (project "sensorboard_DPS310"
-        (path "/ed3d0d35-b5f6-4431-803a-14ff3cdab111"
-          (reference "H1") (unit 1)
         )
       )
@@
     )
   )
-  (symbol (lib_id "Mechanical:MountingHole_Pad") (at 64.77 162.56 0) (unit 1)
-    (in_bom yes) (on_board yes) (dnp no) (fields_autoplaced)
-    (property "Reference" "H2" (at 67.31 160.0779 0)
-      (effects (font (size 1.27 1.27)) (justify left))
-    )
-    (property "Value" "~" (at 67.31 162.5021 0)
-      (effects (font (size 1.27 1.27)) (justify left))
-    )
-    (property "Footprint" "MountingHole:MountingHole_2.2mm_M2_Pad" (at 64.77 162.56 0)
-      (effects (font (size 1.27 1.27)) hide)
-    )
-    (property "Datasheet" "~" (at 64.77 162.56 0)
-      (effects (font (size 1.27 1.27)) hide)
-    )
-    (pin "1")
-    (instances
-      (project "sensorboard_DPS310"
-        (path "/ed3d0d35-b5f6-4431-803a-14ff3cdab111"
-          (reference "H2") (unit 1)
-        )
-      )
-    )
-  )
   (symbol (lib_id "Device:R") (at 208.28 96.52 0) (unit 1)
     (in_bom yes) (on_board yes) (dnp no) (fields_autoplaced)
@@
         )
       )
-    )
-  )
-  (symbol (lib_id "Device:R") (at 121.285 163.83 0) (unit 1)
-    (in_bom no) (on_board yes) (dnp yes) (fields_autoplaced)
-    (property "Reference" "R3" (at 123.063 162.6179 0)
-      (effects (font (size 1.27 1.27)) (justify left))
-    )
-    (property "Value" "10k" (at 123.063 165.0421 0)
-      (effects (font (size 1.27 1.27)) (justify left))
-    )
-    (property "Footprint" "Resistor_SMD:R_0603_1608Metric_Pad0.98x0.95mm_HandSolder" (at 119.507 163.83 90)
-      (effects (font (size 1.27 1.27)) hide)
-    )
-    (property "Datasheet" "~" (at 121.285 163.83 0)
-      (effects (font (size 1.27 1.27)) hide)
-    )
-    (pin "1")
-    (pin "2")
-    (instances
-      (project "sensorboard_DPS310"
-        (path "/ed3d0d35-b5f6-4431-803a-14ff3cdab111"
-          (reference "R3") (unit 1)
-        )
-      )
